Commit message: have a solid planar walking example

File: planar_example/urdf/harpy_planar.urdf (robot description, URDF)
Before this commit: robot harpy, 18 links, 18 joints
Links:
- link FootLeft: geometry collision sphere radius=0.02; visual sphere radius=0.02
- link FootRight: geometry collision sphere radius=0.02; visual sphere radius=0.02
- link SagittalHipLeft: geometry visual mesh filename=../meshes/HipLeft_.obj
- link SagittalHipRight: geometry visual mesh filename=../meshes/HipRight_.obj
- link Torso: geometry collision sphere radius=0.17; visual mesh filename=../meshes/Torso_.obj
